Commit message: New URDF Generated

File: Pallet_Jack/urdf/Pallet_Jack.urdf (robot description, URDF)
Before this commit: robot Pallet_Jack, 6 links, 5 joints
Links:
- link Lidar: mass 1.4060100831482 -> 1.406
- link Steering: mass 44.1786466911065 -> 44.179
- link Wheel: mass 37.6991118430775 -> 37.699
- link Zed_Camera_1: mass 0.615000000000001 -> 0.615
- link Zed_Camera_2: mass 0.615000000000001 -> 0.615
- link base_link: mass 651.526919825643 -> 651.53
