Commit message: src folder split in meshes and urdf

File: pallet_jack_description/urdf/pallet_jack.xacro (robot description, xacro)
@@ -13,5 +13,5 @@
       <origin xyz="0 0 0" rpy="0 0 0" />
       <geometry>
-        <mesh filename="package://pallet_jack_description/src/description/meshes/base_link.STL" />
+        <mesh filename="package://pallet_jack_description/pallet_jack/meshes/base_link.STL" />
       </geometry>
       <material name="">
@@ -22,5 +22,5 @@
       <origin xyz="0 0 0" rpy="0 0 0" />
       <geometry>
-        <mesh filename="package://pallet_jack_description/src/description/meshes/base_link.STL" />
+        <mesh filename="package://pallet_jack_description/pallet_jack/meshes/base_link.STL" />
       </geometry>
     </collision>
@@ -35,5 +35,5 @@
       <origin xyz="0 0 0" rpy="0 0 0" />
       <geometry>
-        <mesh filename="package://pallet_jack_description/src/description/meshes/steering_wheel_link.STL" />
+        <mesh filename="package://pallet_jack_description/pallet_jack/meshes/steering_wheel_link.STL" />
       </geometry>
       <material name="">
@@ -58,5 +58,5 @@
       <origin xyz="0 0 0" rpy="0 0 0" />
       <geometry>
-        <mesh filename="package://pallet_jack_description/src/description/meshes/drive_wheel_link.STL" />
+        <mesh filename="package://pallet_jack_description/pallet_jack/meshes/drive_wheel_link.STL" />
       </geometry>
       <material name="">
@@ -67,5 +67,5 @@
       <origin xyz="0 0 0" rpy="0 0 0" />
       <geometry>
-        <mesh filename="package://pallet_jack_description/src/description/meshes/drive_wheel_link.STL" />
+        <mesh filename="package://pallet_jack_description/pallet_jack/meshes/drive_wheel_link.STL" />
       </geometry>
     </collision>
@@ -87,5 +87,5 @@
       <origin xyz="0 0 0" rpy="0 0 0" />
       <geometry>
-        <mesh filename="package://pallet_jack_description/src/description/meshes/lidar.STL" />
+        <mesh filename="package://pallet_jack_description/pallet_jack/meshes/lidar.STL" />
       </geometry>
       <material name="">
@@ -109,5 +109,5 @@
       <origin xyz="0 0 0" rpy="0 0 0" />
       <geometry>
-        <mesh filename="package://pallet_jack_description/src/description/meshes/zed_cam_1.STL" />
+        <mesh filename="package://pallet_jack_description/pallet_jack/meshes/zed_cam_1.STL" />
       </geometry>
       <material name="">
@@ -131,5 +131,5 @@
       <origin xyz="0 0 0" rpy="0 0 0" />
       <geometry>
-        <mesh filename="package://pallet_jack_description/src/description/meshes/zed_cam_2.STL" />
+        <mesh filename="package://pallet_jack_description/pallet_jack/meshes/zed_cam_2.STL" />
       </geometry>
       <material name="">
@@ -161,5 +161,5 @@
       <origin xyz="0 0 0" rpy="0 0 0" />
       <geometry>
-        <mesh filename="package://pallet_jack_description/src/description/meshes/caster_1.STL" />
+        <mesh filename="package://pallet_jack_description/pallet_jack/meshes/caster_1.STL" />
       </geometry>
       <material name="">
@@ -170,5 +170,5 @@
       <origin xyz="0 0 0" rpy="0 0 0" />
       <geometry>
-        <mesh filename="package://pallet_jack_description/src/description/meshes/caster_1.STL" />
+        <mesh filename="package://pallet_jack_description/pallet_jack/meshes/caster_1.STL" />
       </geometry>
     </collision>
@@ -189,5 +189,5 @@
       <origin xyz="0 0 0" rpy="0 0 0" />
       <geometry>
-        <mesh filename="package://pallet_jack_description/src/description/meshes/caster_2.STL" />
+        <mesh filename="package://pallet_jack_description/pallet_jack/meshes/caster_2.STL" />
       </geometry>
       <material name="">
@@ -198,5 +198,5 @@
       <origin xyz="0 0 0" rpy="0 0 0" />
       <geometry>
-        <mesh filename="package://pallet_jack_description/src/description/meshes/caster_2.STL" />
+        <mesh filename="package://pallet_jack_description/pallet_jack/meshes/caster_2.STL" />
       </geometry>
     </collision>
@@ -217,5 +217,5 @@
       <origin xyz="0 0 0" rpy="0 0 0" />
       <geometry>
-        <mesh filename="package://pallet_jack_description/src/description/meshes/caster_3.STL" />
+        <mesh filename="package://pallet_jack_description/pallet_jack/meshes/caster_3.STL" />
       </geometry>
       <material name="">
@@ -226,5 +226,5 @@
       <origin xyz="0 0 0" rpy="0 0 0" />
       <geometry>
-        <mesh filename="package://pallet_jack_description/src/description/meshes/caster_3.STL" />
+        <mesh filename="package://pallet_jack_description/pallet_jack/meshes/caster_3.STL" />
       </geometry>
     </collision>
@@ -245,5 +245,5 @@
       <origin xyz="0 0 0" rpy="0 0 0" />
       <geometry>
-        <mesh filename="package://pallet_jack_description/src/description/meshes/caster_4.STL" />
+        <mesh filename="package://pallet_jack_description/pallet_jack/meshes/caster_4.STL" />
       </geometry>
       <material name="">
@@ -254,5 +254,5 @@
       <origin xyz="0 0 0" rpy="0 0 0" />
       <geometry>
-        <mesh filename="package://pallet_jack_description/src/description/meshes/caster_4.STL" />
+        <mesh filename="package://pallet_jack_description/pallet_jack/meshes/caster_4.STL" />
       </geometry>
     </collision>

Commit message: tried integrating velodyne lidar in the urdf, but failed.

File: pallet_jack_description/urdf/pallet_jack.xacro (robot description, xacro)
@@ -3,5 +3,5 @@
      Commit Version: 1.6.0-4-g7f85cfe  Build Version: 1.6.7995.38578
      For more information, please see http://wiki.ros.org/sw_urdf_exporter -->
-<robot name="pallet_jack">
+<robot xmlns:xacro="http://ros.org/wiki/xacro" name="pallet_jack">
   <link name="base_link">
     <inertial>
@@ -13,5 +13,5 @@
       <origin xyz="0 0 0" rpy="0 0 0" />
       <geometry>
-        <mesh filename="package://pallet_jack_description/pallet_jack/meshes/base_link.STL" />
+        <mesh filename="package://pallet_jack_description/meshes/base_link.STL" />
       </geometry>
       <material name="">
@@ -22,5 +22,5 @@
       <origin xyz="0 0 0" rpy="0 0 0" />
       <geometry>
-        <mesh filename="package://pallet_jack_description/pallet_jack/meshes/base_link.STL" />
+        <mesh filename="package://pallet_jack_description/meshes/base_link.STL" />
       </geometry>
     </collision>
@@ -35,5 +35,5 @@
       <origin xyz="0 0 0" rpy="0 0 0" />
       <geometry>
-        <mesh filename="package://pallet_jack_description/pallet_jack/meshes/steering_wheel_link.STL" />
+        <mesh filename="package://pallet_jack_description/meshes/steering_wheel_link.STL" />
       </geometry>
       <material name="">
@@ -58,5 +58,5 @@
       <origin xyz="0 0 0" rpy="0 0 0" />
       <geometry>
-        <mesh filename="package://pallet_jack_description/pallet_jack/meshes/drive_wheel_link.STL" />
+        <mesh filename="package://pallet_jack_description/meshes/drive_wheel_link.STL" />
       </geometry>
       <material name="">
@@ -67,5 +67,5 @@
       <origin xyz="0 0 0" rpy="0 0 0" />
       <geometry>
-        <mesh filename="package://pallet_jack_description/pallet_jack/meshes/drive_wheel_link.STL" />
+        <mesh filename="package://pallet_jack_description/meshes/drive_wheel_link.STL" />
       </geometry>
     </collision>
@@ -87,5 +87,5 @@
       <origin xyz="0 0 0" rpy="0 0 0" />
       <geometry>
-        <mesh filename="package://pallet_jack_description/pallet_jack/meshes/lidar.STL" />
+        <mesh filename="package://pallet_jack_description/meshes/lidar.STL" />
       </geometry>
       <material name="">
@@ -109,5 +109,5 @@
       <origin xyz="0 0 0" rpy="0 0 0" />
       <geometry>
-        <mesh filename="package://pallet_jack_description/pallet_jack/meshes/zed_cam_1.STL" />
+        <mesh filename="package://pallet_jack_description/meshes/zed_cam_1.STL" />
       </geometry>
       <material name="">
@@ -131,5 +131,5 @@
       <origin xyz="0 0 0" rpy="0 0 0" />
       <geometry>
-        <mesh filename="package://pallet_jack_description/pallet_jack/meshes/zed_cam_2.STL" />
+        <mesh filename="package://pallet_jack_description/meshes/zed_cam_2.STL" />
       </geometry>
       <material name="">
@@ -161,5 +161,5 @@
       <origin xyz="0 0 0" rpy="0 0 0" />
       <geometry>
-        <mesh filename="package://pallet_jack_description/pallet_jack/meshes/caster_1.STL" />
+        <mesh filename="package://pallet_jack_description/meshes/caster_1.STL" />
       </geometry>
       <material name="">
@@ -170,5 +170,5 @@
       <origin xyz="0 0 0" rpy="0 0 0" />
       <geometry>
-        <mesh filename="package://pallet_jack_description/pallet_jack/meshes/caster_1.STL" />
+        <mesh filename="package://pallet_jack_description/meshes/caster_1.STL" />
       </geometry>
     </collision>
@@ -189,5 +189,5 @@
       <origin xyz="0 0 0" rpy="0 0 0" />
       <geometry>
-        <mesh filename="package://pallet_jack_description/pallet_jack/meshes/caster_2.STL" />
+        <mesh filename="package://pallet_jack_description/meshes/caster_2.STL" />
       </geometry>
       <material name="">
@@ -198,5 +198,5 @@
       <origin xyz="0 0 0" rpy="0 0 0" />
       <geometry>
-        <mesh filename="package://pallet_jack_description/pallet_jack/meshes/caster_2.STL" />
+        <mesh filename="package://pallet_jack_description/meshes/caster_2.STL" />
       </geometry>
     </collision>
@@ -217,5 +217,5 @@
       <origin xyz="0 0 0" rpy="0 0 0" />
       <geometry>
-        <mesh filename="package://pallet_jack_description/pallet_jack/meshes/caster_3.STL" />
+        <mesh filename="package://pallet_jack_description/meshes/caster_3.STL" />
       </geometry>
       <material name="">
@@ -226,5 +226,5 @@
       <origin xyz="0 0 0" rpy="0 0 0" />
       <geometry>
-        <mesh filename="package://pallet_jack_description/pallet_jack/meshes/caster_3.STL" />
+        <mesh filename="package://pallet_jack_description/meshes/caster_3.STL" />
       </geometry>
     </collision>
@@ -245,5 +245,5 @@
       <origin xyz="0 0 0" rpy="0 0 0" />
       <geometry>
-        <mesh filename="package://pallet_jack_description/pallet_jack/meshes/caster_4.STL" />
+        <mesh filename="package://pallet_jack_description/meshes/caster_4.STL" />
       </geometry>
       <material name="">
@@ -254,5 +254,5 @@
       <origin xyz="0 0 0" rpy="0 0 0" />
       <geometry>
-        <mesh filename="package://pallet_jack_description/pallet_jack/meshes/caster_4.STL" />
+        <mesh filename="package://pallet_jack_description/meshes/caster_4.STL" />
       </geometry>
     </collision>
@@ -473,8 +473,8 @@
   <!-- Zed cameras -->
   <!-- Lidar -->
-  <!-- <xacro:include filename="package://velodyne_simulator/veloyne_description/urdf/VLP-16.urdf.xacro"/>
+  <xacro:include filename="package://velodyne_description/urdf/VLP-16.urdf.xacro"/>
   <VLP-16 parent="lidar" name="velodyne" topic="/velodyne_points" hz="10" samples="440" gpu="false">
     <origin xyz="0 0 0" rpy="0 0 0" />
-  </VLP-16> -->
+  </VLP-16>
   <!-- Tricycle Drive -->
 </robot>
